File: PCB/idk.kicad_pcb (KiCad board)
At the start: 2 copper layers, 60.3 x 92.6 mm, 21 parts, among them J1 Conn_01x04_Pin, SW1 SW_Push, SW2 SW_Push, SW3 SW_Push, SW4 SW_Push, SW5 SW_Push, SW6 SW_Push, SW7 SW_Push, SW8 SW_Push, SW9 SW_Push, U1 XIAO-RP2040-DIP

Commit message: tweaks
Parts:
- D10, D2, D3, D4, D5, D6, D7, D8, D9: footprint Diode_SMD:D_SOD-523 -> Dio:D_DO-35_SOD27_P7.62mm_Horizontal
- J1: value Conn_01x04_Pin -> OLED
- renumbered Rotary to SW10
Routing:
- net Net-(D5-A): track 12.3 -> 25.5 mm
- net Net-(D9-A): track 12.2 -> 13.1 mm
- net Net-(D3-A): track 12.4 -> 13.3 mm
- net Net-(D7-A): track 12.4 -> 13.3 mm
- net Net-(D2-A): track 12.4 -> 13.3 mm
- net Net-(D6-A): track 12.4 -> 13.3 mm
- net Net-(D10-A): track 12.4 -> 13.2 mm
- net Net-(D8-A): track 12.5 -> 13.3 mm
- net Net-(D4-A): track 12.5 -> 13.3 mm
