File: PCB/idk.kicad_sch (KiCad schematic)
At the start: 21 parts, among them J1 OLED, SW1 SW_Push, SW10 RotaryEncoder_Switch, SW2 SW_Push, SW3 SW_Push, SW4 SW_Push, SW5 SW_Push, SW6 SW_Push, SW7 SW_Push, SW8 SW_Push, SW9 SW_Push, U1 XIAO-RP2040-DIP

Commit message: tweaks
Parts:
- D10, D2, D3, D4, D5, D6, D7, D8, D9: footprint Diode_SMD:D_SOD-523 -> Dio:D_DO-35_SOD27_P7.62mm_Horizontal
Changed lines of the file:
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@@
 			)
 		)
-		(property "Footprint" "Diode_SMD:D_SOD-523"
+		(property "Footprint" "Dio:D_DO-35_SOD27_P7.62mm_Horizontal"
 			(at 106.045 96.52 0)
 			(effects
@@
 			)
 		)
-		(property "Footprint" "Diode_SMD:D_SOD-523"
+		(property "Footprint" "Dio:D_DO-35_SOD27_P7.62mm_Horizontal"
 			(at 106.045 78.74 0)
 			(effects
@@
 			)
 		)
-		(property "Footprint" "Diode_SMD:D_SOD-523"
+		(property "Footprint" "Dio:D_DO-35_SOD27_P7.62mm_Horizontal"
 			(at 106.045 113.03 0)
 			(effects
@@
 			)
 		)
-		(property "Footprint" "Diode_SMD:D_SOD-523"
+		(property "Footprint" "Dio:D_DO-35_SOD27_P7.62mm_Horizontal"
 			(at 131.445 78.74 0)
 			(effects
@@
 			)
 		)
-		(property "Footprint" "Diode_SMD:D_SOD-523"
+		(property "Footprint" "Dio:D_DO-35_SOD27_P7.62mm_Horizontal"
 			(at 131.445 96.52 0)
 			(effects
@@
 			)
 		)
-		(property "Footprint" "Diode_SMD:D_SOD-523"
+		(property "Footprint" "Dio:D_DO-35_SOD27_P7.62mm_Horizontal"
 			(at 155.575 78.74 0)
 			(effects
@@
 			)
 		)
-		(property "Footprint" "Diode_SMD:D_SOD-523"
+		(property "Footprint" "Dio:D_DO-35_SOD27_P7.62mm_Horizontal"
 			(at 155.575 96.52 0)
 			(effects
@@
 			)
 		)
-		(property "Footprint" "Diode_SMD:D_SOD-523"
+		(property "Footprint" "Dio:D_DO-35_SOD27_P7.62mm_Horizontal"
 			(at 131.445 113.03 0)
 			(effects
@@
 			)
 		)
-		(property "Footprint" "Diode_SMD:D_SOD-523"
+		(property "Footprint" "Dio:D_DO-35_SOD27_P7.62mm_Horizontal"
 			(at 155.575 113.03 0)
 			(effects
